Commit message: Add files via upload

File: diffbot/src/diffbot_description/urdf/ignore_diffbot.xacro (robot description, xacro)
@@ -155,5 +155,5 @@
     <child link="imu_link"/>
   </joint>
-  <link name="camera_rgb_frame">
+  <link name="camera">
     <collision>
       <origin xyz="0 0 0" rpy="0 0 0"/>
@@ -180,5 +180,11 @@
     <origin xyz=".2 0 0" rpy="0 0 0"/>
     <parent link="chassis"/>
-    <child link="camera_rgb_frame"/>
+    <child link="camera"/>
+  </joint>
+  <joint name="hokuyo_joint" type="fixed">
+    <axis xyz="0 1 0" />
+    <origin xyz="0 0 0" rpy="0 0 0"/>
+    <parent link="chassis"/>
+    <child link="hokuyo"/>
   </joint>
   <!-- Hokuyo Laser -->
@@ -191,7 +197,7 @@
     </collision>
     <visual>
-      <origin xyz="0 0 0 " rpy="0 0 0"/>
-      <geometry>
-        <mesh filename="package://$(find diffbot)/src/diffbot_description/meshes/hokuyo.dae"/>
+      <origin xyz="0 0 0" rpy="0 0 0"/>
+      <geometry>
+        <mesh filename="package:$(find diffbot)/src/diffbot_description/urdf/meshes/hokuyo.dae"/>
       </geometry>
     </visual>
@@ -202,9 +208,3 @@
     </inertial>
   </link>
-  <joint name="hokuyo_joint" type="fixed">
-    <axis xyz="0 1 0" />
-    <origin xyz="0.15 0 0.1" rpy="0 0 0"/>
-    <parent link="chassis"/>
-    <child link="hokuyo"/>
-  </joint>
 </robot>

File: diffbot/src/diffbot_description/urdf/ignore_diffbot_gazebo_plugins.xacro (robot description, xacro)
@@ -47,10 +47,9 @@
         <bodyName>imu_link</bodyName>
         <updateRateHZ>10.0</updateRateHZ>
-	<serviceName>imu_service</serviceName>
-	<gaussianNoise>0.0</gaussianNoise>
+        <gaussianNoise>0.0</gaussianNoise>
         <xyzOffset>0 0 0</xyzOffset>
         <rpyOffset>0 0 0</rpyOffset>
         <frameName>imu_link</frameName>
-        <initialOrientationAsReference>false</initialOrientationAsReference>
+        <initialOrientationAsReference>True</initialOrientationAsReference>
       </plugin>
       <pose>0 0 0 0 0 0</pose>
@@ -79,44 +78,33 @@
     <material>Gazebo/Blue</material>
   </gazebo>
-   <gazebo reference="camera_rgb_frame">
-    <sensor type="depth" name="realsense_R200">
-      <always_on>true</always_on>
-      <material>Gazebo/Green</material>
-      <camera>
-          <horizontal_fov>1.3439</horizontal_fov>
-          <image>
-              <width>1920</width>
-              <height>1080</height>
-              <format>R8G8B8</format>
-          </image>
-          <depth_camera></depth_camera>
-          <clip>
-              <near>0.03</near>
-              <far>100</far>
-          </clip>
+  <gazebo reference="camera">
+    <material>Gazebo/Green</material>
+    <sensor type="camera" name="camera1">
+      <update_rate>30.0</update_rate>
+      <camera name="head">
+        <horizontal_fov>1.3962634</horizontal_fov>
+        <image>
+          <width>800</width>
+          <height>800</height>
+          <format>R8G8B8</format>
+        </image>
+        <clip>
+          <near>0.02</near>
+          <far>300</far>
+        </clip>
       </camera>
-      <plugin name="camera_controller" filename="libgazebo_ros_openni_kinect.so">
-        <baseline>0.2</baseline>
+      <plugin name="camera_controller" filename="libgazebo_ros_camera.so">
         <alwaysOn>true</alwaysOn>
-        <updateRate>45.0</updateRate>
-        <cameraName>camera</cameraName>
-        <frameName>camera_rgb_frame</frameName>
-        <imageTopicName>rgb/image_raw</imageTopicName>
-        <depthImageTopicName>depth_registered/image_raw</depthImageTopicName>
-        <pointCloudTopicName>depth/points</pointCloudTopicName>
-        <cameraInfoTopicName>rgb/camera_info</cameraInfoTopicName>
-        <depthImageCameraInfoTopicName>depth/camera_info</depthImageCameraInfoTopicName>
-        <pointCloudCutoff>0.4</pointCloudCutoff>
-            <hackBaseline>0.07</hackBaseline>
-            <distortionK1>0.0</distortionK1>
-            <distortionK2>0.0</distortionK2>
-            <distortionK3>0.0</distortionK3>
-            <distortionT1>0.0</distortionT1>
-            <distortionT2>0.0</distortionT2>
-        <CxPrime>0.0</CxPrime>
-        <Cx>0.0</Cx>
-        <Cy>0.0</Cy>
-        <focalLength>0</focalLength>
-        <hackBaseline>0</hackBaseline>
+        <updateRate>0.0</updateRate>
+        <cameraName>diffbot_camera1</cameraName>
+        <imageTopicName>image_raw</imageTopicName>
+        <cameraInfoTopicName>camera_info</cameraInfoTopicName>
+        <frameName>camera</frameName>
+        <hackBaseline>0.07</hackBaseline>
+        <distortionK1>0.0</distortionK1>
+        <distortionK2>0.0</distortionK2>
+        <distortionK3>0.0</distortionK3>
+        <distortionT1>0.0</distortionT1>
+        <distortionT2>0.0</distortionT2>
       </plugin>
     </sensor>
@@ -126,6 +114,6 @@
     <sensor type="gpu_ray" name="head_hokuyo_sensor">
       <pose>0 0 0 0 0 0</pose>
-      <visualize>true</visualize>
-      <update_rate>45</update_rate>
+      <visualize>false</visualize>
+      <update_rate>40</update_rate>
       <ray>
         <scan>
@@ -153,5 +141,5 @@
       </ray>
       <plugin name="gazebo_ros_head_hokuyo_controller" filename="libgazebo_ros_gpu_laser.so">
-        <topicName>/diffbot/laser_scan</topicName>
+        <topicName>diffbot_laser_scan</topicName>
         <frameName>hokuyo</frameName>
       </plugin>
